File: PCB/Junco.kicad_sch (KiCad schematic)
At the start: 202 parts, among them J1 AudioJack4, J2 AudioJack4, SW1 SW_Push, SW10 SW_Push, SW11 SW_Push, SW12 SW_Push, SW13 SW_Push, SW14 SW_Push, SW15 SW_Push, SW16 SW_Push, SW17 SW_Push, SW18 SW_Push, SW19 SW_MX_Hotswap_Rotary, SW2 SW_Push, SW20 SW_Push, SW21 SW_Push, SW22 SW_Push, SW23 SW_Push, SW24 SW_Push, SW25 SW_Push, SW26 SW_Push, SW27 SW_Push, SW28 SW_Push, SW29 SW_Push, SW3 SW_Push, SW30 RotaryEncoder_Switch, SW31 SW_Push, SW32 SW_Push, SW33 SW_Push, SW34 SW_Push, SW35 SW_Push, SW36 SW_Push, SW37 SW_Push, SW38 SW_Push, SW39 SW_Push, SW4 SW_Push, SW40 SW_Push, SW41 SW_Push, SW42 SW_Push, SW43 SW_Push, SW44 SW_Push, SW45 SW_Push, SW46 SW_Push, SW47 SW_Push, SW48 SW_Push, SW49 SW_MX_Hotswap_Rotary, SW5 SW_Push, SW50 SW_Push, SW51 SW_Push, SW52 SW_Push, SW53 SW_Push, SW54 SW_Push, SW55 SW_Push, SW56 SW_Push, SW57 SW_Push, SW58 SW_Push, SW59 SW_Push, SW6 SW_Push, SW60 RotaryEncoder_Switch, SW7 SW_Push, SW8 SW_Push, SW9 SW_Push, U1 Pico, U2 SN74AHCT1G125, U3 Pico, U4 SN74AHCT1G125

Commit message: Key rotation & other QOL improvements (#2)
* Keycap rotation
Swapped in smd/through-hole diode footprints

* comitt before pcb led rotation unification
already updated LED orientation on schematic

* Finished main led flip
underglow flip remains

* Added hardware 'handedness on gp18 with default LH

* Updated corner encoders
Created flipped encoder/switch combo footprint
Created short offset LED for encoder/switch combo
Encoder routing
Added build notes

* Wiring cleanup

* Routing cleanup

* Routing cleanup

* Removed LED legs and cleaned up routing

* DRC unconnected item repair

* Alined diode orientation
updated routing for modified diodes
Updated diode labeling

* Removed nested clone

* Added fiducials

* Cleanup for fab
switched Diode sides in footprint then on board so it would appear on bottom pos
changed pico & rotary encoder component type to fix DRC error
generated gerbers
generated bom
generated pos

* Flipped LED footrpints for placement file

* Updated footprints to exclude through-hole components from position files

* Added JLC part number to LED and switch symbols

* DRC rules updated with JLC specs
Imported specs from https://github.com/sethhillbrand/kicad_templates
Fixed all rule violations
increased default vias
minor trace cleanup

* Updated minimum annular width
Updated copper to edge param
updated board accordingly

* Updated copper to hole and hole to hole
updated routing accordingly
adjusted LED tracks for new via size

* Moved vias off smd pads

* Added level shifter bypass jumper
Schematic updated
Symbol created and placed

* Culled unused footprints

* Moved under-glow LED's to top side for PNP placement

* Fixed Rotary/switch combo footprint orientation for PNP placement

* Added JLC part numbers to BOM

* Consolidated LED footprints

* Consolidated Switch footprints with 1.5u and 1u

* Updated BOM & PNP

* Updated SK6803 footprint to match tape reel orien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
Parts:
- added FID1, FID2, FID3, FID4: Fiducial, Fiducial:Fiducial_1mm_Mask2mm, symbol Mechanical:Fiducial
- added JP1, JP2: Level shifter bypass jumper, Junco:Level Shifter Bypass Jumper, symbol Jumper:SolderJumper_2_Open
- D1, D10, D11, D12, D13, D14, D15, D16, D17, D18, D19, D2, D20, D21, D22, D23, D24, D25, D26, D27, D28, D29, D3, D30, D31, D32, D33, D34, D35, D36, D37, D38, D39, D4, D40, D41, D42, D43, D44, D45, D46, D47, D48, D49, D5, D50, D51, D52, D53, D54, D55, D56, D57, D58, D59, D6, D60, D61, D62, D7, D8, D9: footprint Junco:D_SOD-123 -> Junco:D_SOD-123_DO-35_Hybrid_DoubleSided_V2
- SK68XX_Mini1, SK68XX_Mini2, SK68XX_Mini3, SK68XX_Mini38, SK68XX_Mini39, SK68XX_Mini4, SK68XX_Mini40, SK68XX_Mini41, SK68XX_Mini42, SK68XX_Mini43, SK68XX_Mini44, SK68XX_Mini45, SK68XX_Mini5, SK68XX_Mini6, SK68XX_Mini7, SK68XX_Mini8: value SK68XXMini -> SK6803MINI-E; footprint Junco:SK68XXMini -> Junco:SK68XXMini_drill_hole_mod
- SK68XX_Mini10, SK68XX_Mini11, SK68XX_Mini12, SK68XX_Mini13, SK68XX_Mini14, SK68XX_Mini21, SK68XX_Mini22, SK68XX_Mini23, SK68XX_Mini24, SK68XX_Mini25, SK68XX_Mini26, SK68XX_Mini35, SK68XX_Mini36, SK68XX_Mini37, SK68XX_Mini52, SK68XX_Mini53, SK68XX_Mini54, SK68XX_Mini55, SK68XX_Mini56, SK68XX_Mini57, SK68XX_Mini64, SK68XX_Mini65, SK68XX_Mini66, SK68XX_Mini67, SK68XX_Mini68, SK68XX_Mini69, SK68XX_Mini70, SK68XX_Mini71, SK68XX_Mini9: value SK68XXMini -> SK6803MINI-E; footprint Junco:SK68XXMini_Offset_Flipped -> Junco:SK68XXMini_drill_hole_mod
- SK68XX_Mini15, SK68XX_Mini16, SK68XX_Mini17, SK68XX_Mini18, SK68XX_Mini19, SK68XX_Mini20, SK68XX_Mini27, SK68XX_Mini28, SK68XX_Mini29, SK68XX_Mini30, SK68XX_Mini31, SK68XX_Mini32, SK68XX_Mini33, SK68XX_Mini34, SK68XX_Mini46, SK68XX_Mini47, SK68XX_Mini48, SK68XX_Mini49, SK68XX_Mini50, SK68XX_Mini51, SK68XX_Mini58, SK68XX_Mini59, SK68XX_Mini60, SK68XX_Mini61, SK68XX_Mini62, SK68XX_Mini63, SK68XX_Mini72, SK68XX_Mini73, SK68XX_Mini74: value SK68XXMini -> SK6803MINI-E; footprint Junco:SK68XXMini_Offset -> Junco:SK68XXMini_drill_hole_mod
- SW19, SW49: value SW_MX_Hotswap_Rotary -> SW_MX_Hotswap_Rotary_Switch; footprint Junco:SW_MX_Hotswap_Rotary -> Junco:SW_MX_Hotswap_Rotary_Switch
- SW28, SW29, SW58, SW59: footprint marbast_mx:SW_MX_HS_1.5u -> marbast_mx:SW_MX_HS_1u
Connections:
- net GNDA: now also U3.24 (GPIO18)
- net VCC: now also U1.24 (GPIO18)
- net led: now also JP1.1 (A)
- net led_r: now also JP2.1 (A)
- net at SK68XX_Mini38.4 (DIN), U4.4 (DOUT): now also JP2.2 (B)
- net at SK68XX_Mini1.4 (DIN), U2.4 (DOUT): now also JP1.2 (B)
- no-connect marks 42 -> 40
Other:
- note added: "Pulled high for handedness"
- note added: "Pulled low for handedness"
- note added: "Used for component placement"
- moved on the sheet: SK68XX_Mini1, SK68XX_Mini10, SK68XX_Mini11, SK68XX_Mini12, SK68XX_Mini13, SK68XX_Mini14, SK68XX_Mini15, SK68XX_Mini16, SK68XX_Mini17, SK68XX_Mini18, SK68XX_Mini19, SK68XX_Mini2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
